File: printer-expasion.kicad_pcb (KiCad board)
At the start: 2 copper layers, 95 x 75 mm, 80 parts, among them J1 Screw_Terminal_DC_input, J10 pinda1, J11 pinda2, J12 pinda3, J13 Conn_02x04_Odd_Even, J14 fan, J15 fan, J16 fan, J17 fan, J18 Conn_02x04_Odd_Even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

Commit message: get shrunk
Parts:
- moved H4 42.0 mm to (137.0, 64.0)
- moved J1 35.8 mm to (180.0, 110.0)
- moved H2 31.9 mm to (195.0, 109.5)
- moved JP1 30.3 mm to (177.5, 86.8), turned to -90 degrees
- moved F1 29.0 mm to (185.0, 90.3), turned to -90 degrees
- moved J10 27.6 mm to (171.5, 95.0)
- moved J11 18.5 mm to (171.6, 100.0)
- moved J19 15.9 mm to (171.5, 110.0)
- moved J12 13.1 mm to (171.6, 105.0)
- moved H1 7.50 mm to (137.0, 109.5)
Routing:
- net pinda4: track 114.9 -> 77.8 mm, vias 2 -> 1
- net +5V: track 254.1 -> 219.8 mm, vias 9 -> 6
- net pinda3: track 78.4 -> 44.9 mm
- net pinda2: track 69.1 -> 40.4 mm
- net pinda1: track 58.6 -> 35.3 mm
- net +3.3V: track 308.5 -> 300.9 mm, vias 12 -> 11
- net Net-(J1-Pin_1): track 23.1 -> 26.9 mm
- net +24V: track 175.1 -> 176.5 mm, vias 4 -> 6
- net Net-(J5-Pin_6): track 17.8 -> 16.4 mm
- net Net-(J5-Pin_4): track 13.0 -> 12.2 mm
- net Net-(J3-Pin_3): track 5.90 -> 5.18 mm
- net GND: track 73.2 -> 73.0 mm, vias 19 -> 22
Other:
- board size 95 x 75 mm -> 95 x 67.5 mm

Commit message: final
Parts:
- removed TP1, TP10, TP11, TP12, TP2, TP3, TP4, TP5, TP6, TP7, TP8, TP9: TestPoint, TestPoint:TestPoint_THTPad_1.0x1.0mm_Drill0.5mm
- added J20: vhdl conn, Connector_PinHeader_2.54mm:PinHeader_2x04_P2.54mm_Vertical, F.Cu at (189.5, 82.1)
- added J21: motor 3, Connector_PinHeader_2.54mm:PinHeader_1x04_P2.54mm_Vertical, F.Cu at (183.0, 90.5)
- added JP21: bypass, Jumper:SolderJumper-2_P1.3mm_Open_Pad1.0x1.5mm, F.Cu at (141.5, 64.2)
- JP10, JP11, JP2, JP3, JP4, JP6, JP7, JP8, JP9: footprint Jumper:SolderJumper-3_P1.3mm_Open_Pad1.0x1.5mm -> Connector_PinHeader_2.54mm:PinHeader_1x03_P2.54mm_Vertical
- moved J4 20.1 mm to (211.4, 66.3)
- moved J6 19.0 mm to (211.0, 87.0)
- moved A2 17.9 mm to (217.6, 91.4), turned to 180 degrees
- moved A1 17.9 mm to (217.7, 68.9), turned to 180 degrees
- moved F1 15.1 mm to (194.7, 102.0), turned to 180 degrees
- moved JP11 14.3 mm to (203.0, 105.0), turned to 90 degrees
- moved JP2 13.9 mm to (208.9, 61.3), turned to 90 degrees
- moved JP8 12.1 mm to (209.0, 82.0), turned to 90 degrees
- moved JP4 12.0 mm to (208.8, 51.3), turned to 90 degrees
- moved JP6 12.0 mm to (209.0, 74.0), turned to 90 degrees
- moved JP3 10.9 mm to (208.8, 56.3), turned to 90 degrees
- moved JP7 10.2 mm to (209.0, 78.0), turned to 90 degrees
- moved J8 9.62 mm to (207.0, 101.0)
- moved J7 9.50 mm to (225.0, 87.5), turned to 180 degrees
- moved JP10 9.39 mm to (219.0, 101.0), turned to -90 degrees
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Connections:
- U1 pad 11: en3 -> dir3
- U1 pad 23: +5V -> Net-(JP21-A)
- U1 pad 3: dir1 -> en1
- U1 pad 5: en1 -> dir1
- U1 pad 6: dir2 -> en2
- U1 pad 8: en2 -> dir2
- U1 pad 9: dir3 -> en3
Routing:
- net +5V: track 219.8 -> 171.9 mm, vias 6 -> 4
- net Net-(JP21-A): track 0.00 -> 45.3 mm, vias 0 -> 2
- net step1: track 14.2 -> 53.1 mm
- net dir2: track 20.4 -> 54.8 mm
- net dir1: track 15.4 -> 47.6 mm
- net step2: track 23.7 -> 55.6 mm
- net en1: track 28.9 -> 56.3 mm
- net en2: track 36.8 -> 57.0 mm
- net Net-(A1-1B): track 27.3 -> 7.84 mm
- net Net-(A2-1B): track 27.1 -> 7.90 mm
- net +3.3V: track 300.9 -> 283.3 mm
- net Net-(A1-1A): track 23.3 -> 7.84 mm
- net Net-(A2-1A): track 23.1 -> 7.90 mm
- net +24V: track 176.5 -> 190.5 mm, vias 6 -> 5
- net Net-(A1-2A): track 19.4 -> 7.84 mm
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Other:
- board size 95 x 67.5 mm -> 95 x 67 mm
- board text added: "10K R"
- board text added: "3V3"
- board text added: "3v3"
- board text added: "5V-gnd-24V"
- board text added: "5v rx tx gnd"
- board text added: "<=== short for USB power"
- board text added: "GND"
- board text added: "PINDA"
- board text added: "b1 b2 b3 b4"
- board text added: "dir1"
- board text added: "dir2"
- board text added: "en1"
- board text added: "en2"
- board text added: "fan1 - +"
- board text added: "fan2 - +"
- board text added: "fan3 - +"
- board text added: "fan4 - +"
- board text added: "gnd"
- board text added: "p1"
- board text added: "p2"
- board text added: "p3"
- board text added: "p4"
- board text added: "prb-black GND-blue 5V -brown"
- board text added: "rusz.space base48.cz vega76.cz"
- board text added: "step1"
- board text added: "step2"
- board text added: "triple extruder klipper board v0.1 - 2024"
